File: split-choc-z-board/split-choc-z-board-left.kicad_sch (KiCad schematic)
At the start: 44 parts, among them J1 AudioJack4_Ground, SW1 SW_SPST, SW10 SW_SPST, SW11 SW_SPST, SW12 SW_SPST, SW13 SW_SPST, SW14 SW_SPST, SW15 SW_SPST, SW16 SW_SPST, SW17 SW_SPST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

Commit message: Refactored schematic and added footprint library
Parts:
- removed A1: Arduino_Nano_Every, Module:Arduino_Nano, symbol MCU_Module:Arduino_Nano_Every
- removed D1, D10, D11, D12, D13, D14, D15, D16, D17, D18, D2, D3, D4, D5, D6, D7, D8, D9: D, symbol Device:D
- removed J1: AudioJack4_Ground, symbol Connector_Audio:AudioJack4_Ground
- removed R1, R2: 2.2k, symbol Device:R
- removed R3, R4, R5, R6: R, symbol Device:R
- removed SW1, SW10, SW11, SW12, SW13, SW14, SW15, SW16, SW17, SW18, SW2, SW3, SW4, SW5, SW6, SW7, SW8, SW9: SW_SPST, symbol Switch:SW_SPST
Other:
- note removed: "I2C Pull-up resistors"
- note removed: "Keyboard matrix"
- note removed: "Pull-up resistors"
- note removed: "TTRS Connector"
- note removed: "Use this in QMK: #define SPLIT_HAND_PIN A0 HIGH is left hand"
