File: split-choc-z-board-right/split-choc-z-board.kicad_sch (KiCad schematic)
At the start: 45 parts, among them J1 USB4105-GF-A, SW1 SW_SPST, SW10 SW_SPST, SW11 SW_SPST, SW12 SW_SPST, SW13 SW_SPST, SW14 SW_SPST, SW15 SW_SPST, SW16 SW_SPST, SW17 SW_SPST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

Commit message: Finished routing right side! 🤖
Changed lines of the file:
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@@
+	)
+	(junction
+		(at 182.88 63.5)
+		(diameter 0)
+		(color 0 0 0 0)
 	)
 	(junction
@@
 	(wire
 		(pts
-			(xy 205.74 63.5) (xy 180.34 63.5)
+			(xy 205.74 63.5) (xy 182.88 63.5)
 		)
 		(stroke
@@
 	(wire
 		(pts
+			(xy 182.88 63.5) (xy 180.34 63.5)
+		)
+		(stroke
+			(width 0)
+			(type default)
+		)
+	)
+	(wire
+		(pts
 			(xy 205.74 104.14) (xy 205.74 114.3)
 		)
@@
 		(pts
 			(xy 274.32 53.34) (xy 274.32 78.74)
+		)
+		(stroke
+			(width 0)
+			(type default)
+		)
+	)
+	(wire
+		(pts
+			(xy 182.88 60.96) (xy 182.88 63.5)
 		)
 		(stroke
@@
 	)
 	(label "Row 1"
-		(at 182.88 63.5 0)
+		(at 182.88 60.96 0)
 		(effects
 			(font
