File: split-choc-z-board-right/split-choc-z-board.kicad_pcb (KiCad board)
At the start: 2 copper layers, 147.1 x 106.5 mm, 79 parts, among them J1 USB4105-GF-A, J2 USB4105-GF-A, J3 Conn_01x04_Pin, J4 Conn_01x02, SW1 SW_SPST, SW10 SW_SPST, SW11 SW_SPST, SW12 SW_SPST, SW13 SW_SPST, SW14 SW_SPST, SW15 SW_SPST, SW16 SW_SPST, SW17 SW_SPST, SW18 SW_SPST, SW19 SW_SPST, SW2 SW_SPST, SW20 SW_SPST, SW21 SW_SPST, SW22 SW_SPST, SW3 SW_SPST, SW4 SW_SPST, SW5 SW_SPST, SW6 SW_SPST, SW7 SW_SPST, SW8 SW_SPST, SW9 SW_SPST, U2 RP2040, U3 NCP1117-3.3_SOT223, U4 W25Q128JVS, U5 USBLC6-2SC6, X1 ABM8-272-T3

Commit message: Added name and date to board 2
Other:
- board text added: "Zain Kergaye 6/24/25"
Changed lines of the file:
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@@
 		(layer "Edge.Cuts")
+	)
+	(gr_text "Zain Kergaye\n6/24/25"
+		(at 46.725 57.675 90)
+		(layer "F.SilkS")
+		(effects
+			(font
+				(size 1 1)
+				(thickness 0.1)
+			)
+			(justify left bottom)
+		)
 	)
 	(segment
